File: Project_Gmic.sch (KiCad schematic (older format))
At the start: 50 parts, among them J1 USB4085-GF-A, J2 SJ1-3523N, SW1 SW_SPDT, U1 MCP6479, U2 MCP6476U, U3 MCP6476U, U4 XC6351A120MR-G

Commit message: BOM, finishing PCB, changing some non-available components
Parts:
- removed U2, U3: MCP6476U, Package_TO_SOT_SMD:SOT-23-5, symbol Custom:MCP6476U
- removed U4: XC6351A120MR-G, Package_TO_SOT_SMD:SOT-23-6_Handsoldering, symbol Custom:XC6351A120MR-G
- added C21: NC, Capacitor_SMD:C_0805_2012Metric, symbol Device:C
- added U2, U3: AD8531, Package_TO_SOT_SMD:SOT-23-5, symbol Custom:AD8531
- added U4: MAX1852, Package_TO_SOT_SMD:SOT-363_SC-70-6_Handsoldering, symbol Custom:MAX1852
- R1, R2: value 2k2 -> 2.2k
- SW1: value SW_SPDT -> PCM12SMTR
Connections:
- net +5V: now also U2.5 (V+), U3.5 (V+), U4.4 (Vin)
- net -5V: now also U2.2 (V-), U3.2 (V-), U4.1 (Vout)
- net AUDIO_AVERAGE: now also U2.1
- net AUDIO_OUT: now also U3.1
- net GND: now also U4.2 (GND), U4.3 (~SHDN)
- net GNDA: now also U2.3 (+), U3.3 (+)
- net at R6.1, R7.1, R9.2: now also U2.4 (-)
- net at R14.1, R15.2: now also U3.4 (-)
- net at C15.1: now also U4.6 (C1+)
- net at C15.2: now also U4.5 (C1-)
- net at SW1.2 (B): now also C21.2; no longer J2.2
- new net: C21.1, J2.2
Changed lines of the file:
@@
 Last amplification
-$Comp
-L Custom:XC6351A120MR-G U4
-U 1 1 5EE1D5B0
-P 10050 4550
-F 0 "U4" H 10050 5017 50  0000 C CNN
-F 1 "XC6351A120MR-G" H 10050 4926 50  0000 C CNN
-F 2 "Package_TO_SOT_SMD:SOT-23-6_Handsoldering" H 9650 4850 50  0001 C CNN
-F 3 "" H 9650 4850 50  0001 C CNN
-	1    10050 4550
-	1    0    0    -1
-$EndComp
 $Comp
 L power:GND #PWR0112
@@
 P 750 1150
 F 0 "R1" H 820 1196 50  0000 L CNN
-F 1 "2k2" H 820 1105 50  0000 L CNN
+F 1 "2.2k" H 820 1105 50  0000 L CNN
 F 2 "Resistor_SMD:R_0805_2012Metric" V 680 1150 50  0001 C CNN
 F 3 "~" H 750 1150 50  0001 C CNN
@@
 P 1800 1150
 F 0 "R2" H 1870 1196 50  0000 L CNN
-F 1 "2k2" H 1870 1105 50  0000 L CNN
+F 1 "2.2k" H 1870 1105 50  0000 L CNN
 F 2 "Resistor_SMD:R_0805_2012Metric" V 1730 1150 50  0001 C CNN
 F 3 "~" H 1800 1150 50  0001 C CNN
@@
 Wire Wire Line
 	5050 5200 5050 5400
-$Comp
-L Custom:MCP6476U U2
-U 1 1 6225817D
-P 4100 3150
-F 0 "U2" H 4100 3450 50  0000 L CNN
-F 1 "MCP6476U" H 4100 3350 50  0000 L CNN
-F 2 "Package_TO_SOT_SMD:SOT-23-5" H 4450 2750 50  0001 C CNN
-F 3 "https://ww1.microchip.com/downloads/en/DeviceDoc/MCP6476-6R-6U-7-9-Data-Sheet-20006419B.pdf" H 4450 2750 50  0001 C CNN
-	1    4100 3150
-	1    0    0    -1
-$EndComp
 Wire Wire Line
 	4050 3550 3750 3550
@@
 Wire Wire Line
 	4350 3550 4450 3550
-Wire Wire Line
-	4450 3550 4450 3150
 Connection ~ 4450 3150
 Wire Wire Line
@@
 Wire Wire Line
 	3550 3050 3550 3450
-$Comp
-L Custom:MCP6476U U3
-U 1 1 622DA264
-P 7200 3100
-F 0 "U3" H 7200 3400 50  0000 L CNN
-F 1 "MCP6476U" H 7200 3300 50  0000 L CNN
-F 2 "Package_TO_SOT_SMD:SOT-23-5" H 7550 2700 50  0001 C CNN
-F 3 "https://ww1.microchip.com/downloads/en/DeviceDoc/MCP6476-6R-6U-7-9-Data-Sheet-20006419B.pdf" H 7550 2700 50  0001 C CNN
-	1    7200 3100
-	1    0    0    -1
-$EndComp
 Wire Wire Line
 	3300 4450 4050 4450
@@
 P 9550 3100
 F 0 "SW1" H 9550 3385 50  0000 C CNN
-F 1 "SW_SPDT" H 9550 3294 50  0000 C CNN
+F 1 "PCM12SMTR" H 9550 3294 50  0000 C CNN
 F 2 "Button_Switch_SMD:SW_SPDT_PCM12" H 9550 3100 50  0001 C CNN
 F 3 "~" H 9550 3100 50  0001 C CNN
@@
 	9300 3450 10450 3450
 Wire Wire Line
-	9750 3100 10250 3100
+	9750 3100 9850 3100
 $Comp
 L power:GNDA #PWR0125
@@
 	1    0    0    -1
 $EndComp
+$Comp
+L Device:C C21
+U 1 1 62855F87
+P 10000 3100
+F 0 "C21" V 9748 3100 50  0000 C CNN
+F 1 "NC" V 9839 3100 50  0000 C CNN
+F 2 "Capacitor_SMD:C_0805_2012Metric" H 10038 2950 50  0001 C CNN
+F 3 "~" H 10000 3100 50  0001 C CNN
+	1    10000 3100
+	0    1    1    0
+$EndComp
+Wire Wire Line
+	10150 3100 10250 3100
+$Comp
+L Custom:MAX1852 U4
+U 1 1 62892AF9
+P 10050 4550
+F 0 "U4" H 10050 5017 50  0000 C CNN
+F 1 "MAX1852" H 10050 4926 50  0000 C CNN
+F 2 "Package_TO_SOT_SMD:SOT-363_SC-70-6_Handsoldering" H 9650 4850 50  0001 C CNN
+F 3 "" H 9650 4850 50  0001 C CNN
+	1    10050 4550
+	1    0    0    -1
+$EndComp
+$Comp
+L Custom:AD8531 U2
+U 1 1 628EF8E2
+P 4100 3150
+F 0 "U2" H 4150 3400 50  0000 L CNN
+F 1 "AD8531" H 4150 3300 50  0000 L CNN
+F 2 "Package_TO_SOT_SMD:SOT-23-5" H 4450 2750 50  0001 C CNN
+F 3 "https://www.mouser.ch/datasheet/2/609/AD8531_8532_8534-1502287.pdf" H 4450 2750 50  0001 C CNN
+	1    4100 3150
+	1    0    0    -1
+$EndComp
+Wire Wire Line
+	4450 3150 4450 3550
+$Comp
+L Custom:AD8531 U3
+U 1 1 6290E884
+P 7200 3100
+F 0 "U3" H 7250 3350 50  0000 L CNN
+F 1 "AD8531" H 7250 3250 50  0000 L CNN
+F 2 "Package_TO_SOT_SMD:SOT-23-5" H 7550 2700 50  0001 C CNN
+F 3 "https://www.mouser.ch/datasheet/2/609/AD8531_8532_8534-1502287.pdf" H 7550 2700 50  0001 C CNN
+	1    7200 3100
+	1    0    0    -1
+$EndComp
