File: fileFilteringAndAmplification.kicad_sch (KiCad schematic)
At the start: 31 parts, among them U3 AD8532, U4 AD8532, U5 AD8532, U6 AD8531

Commit message: placement, BOM inside kicad
Parts:
- C15, C17: footprint Capacitor_SMD:C_0805_2012Metric -> Capacitor_SMD:C_1206_3216Metric; Manufacturer (none) -> Murata Electronics; Price (none) -> 0.898; Store (none) -> Mouser; StoreID (none) -> 81-GRT31C5C1H104FA2L
- C16, C18, C19: Manufacturer (none) -> Murata Electronics; Price (none) -> 0.381; Store (none) -> Mouser; StoreID (none) -> 81-GCM2165C1H101FA6D
- C20: value 2.2uF -> 2.2uF 16V X7R; Manufacturer (none) -> Samsung Electro-Mechanics; Price (none) -> 0.109; Store (none) -> Mouser; StoreID (none) -> 187-CL21B225KOFNNNE
- C21, C23, C25, C27: Manufacturer (none) -> Wurth Elektronik; Price (none) -> 0.053; Store (none) -> Mouser; StoreID (none) -> 710-885012207045
- C22, C24, C26, C28: Manufacturer (none) -> Wurth Elektronik; Price (none) -> 0.091; Store (none) -> Mouser; StoreID (none) -> 710-885012207051
- R10, R13, R14, R16, R7: Manufacturer (none) -> Panasonic; Price (none) -> 0.091; Store (none) -> Mouser; StoreID (none) -> 667-ERJ-6ENF8062V
- R11, R12, R8, R9: Manufacturer (none) -> Panasonic; Price (none) -> 0.091; Store (none) -> Mouser; StoreID (none) -> 667-ERJ-6ENF1003V
- R15: Manufacturer (none) -> Panasonic; Price (none) -> 0.091; Store (none) -> Mouser; StoreID (none) -> 667-ERJ-6ENF4992V
- R17, R18: Manufacturer (none) -> Panasonic; Price (none) -> 0.099; Store (none) -> Mouser; StoreID (none) -> 667-ERJ-6ENF1002V
- RV1: Manufacturer (none) -> Bourns; Price (none) -> 0.975; Store (none) -> Mouser; StoreID (none) -> 652-PTV09A-4020FA504
- U3, U4, U5: Manufacturer (none) -> Analog Devices; Price (none) -> 1.83; Store (none) -> Mouser; StoreID (none) -> 584-AD8532ARZ-R7
- U6: Manufacturer (none) -> Analog Devices; Price (none) -> 1.43; Store (none) -> Mouser; StoreID (none) -> 584-AD8531ARTZ-R
